File: workshop-5-1/kicad/kicad.kicad_sch (KiCad schematic)
At the start: 36 parts, among them CN1 XH-2AW, SW1 GT-TC060A, SW2 GT-TC060A, SW3 JS102011SAQN, U1 ESP32-S3-WROOM-1-N16R8, U5 BQ24040DSQR, U6 TLV75801PDBVR

Commit message: workshop-5-2
Parts:
- U5: footprint workshop:WSON-10-1EP_2x2mm_P0.4mm_EP0.9x1.5mm -> Package_SON:WSON-10-1EP_2.5x2.5mm_P0.5mm_EP1.2x2mm
Changed lines of the file:
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@@
 		(color 0 0 0 0)
 	)
+	(junction
+		(at 66.04 207.01)
+		(diameter 0)
+		(color 0 0 0 0)
+	)
+	(no_connect
+		(at 50.8 218.44)
+	)
 	(no_connect
 		(at 59.69 73.66)
@@
 	(wire
 		(pts
+			(xy 190.5 243.84) (xy 190.5 251.46)
+		)
+		(stroke
+			(width 0)
+			(type default)
+		)
+	)
+	(wire
+		(pts
+			(xy 163.83 251.46) (xy 163.83 243.84)
+		)
+		(stroke
+			(width 0)
+			(type default)
+		)
+	)
+	(wire
+		(pts
 			(xy 59.69 45.72) (xy 76.2 45.72)
 		)
@@
 	(wire
 		(pts
-			(xy 190.5 243.84) (xy 190.5 251.46)
+			(xy 190.5 228.6) (xy 173.99 228.6)
 		)
 		(stroke
@@
 	(wire
 		(pts
-			(xy 190.5 251.46) (xy 163.83 251.46)
+			(xy 190.5 233.68) (xy 184.15 233.68)
 		)
 		(stroke
@@
 	(wire
 		(pts
-			(xy 163.83 251.46) (xy 163.83 243.84)
+			(xy 190.5 238.76) (xy 186.69 238.76)
 		)
 		(stroke
@@
 	(wire
 		(pts
-			(xy 190.5 228.6) (xy 173.99 228.6)
+			(xy 215.9 228.6) (xy 228.6 228.6)
 		)
 		(stroke
@@
 	(wire
 		(pts
-			(xy 190.5 233.68) (xy 184.15 233.68)
+			(xy 215.9 238.76) (xy 219.71 238.76)
 		)
 		(stroke
@@
 	(wire
 		(pts
-			(xy 190.5 238.76) (xy 186.69 238.76)
+			(xy 219.71 238.76) (xy 219.71 251.46)
 		)
 		(stroke
@@
 	(wire
 		(pts
-			(xy 215.9 228.6) (xy 228.6 228.6)
+			(xy 203.2 255.27) (xy 203.2 257.81)
 		)
 		(stroke
@@
 	(wire
 		(pts
-			(xy 215.9 238.76) (xy 219.71 238.76)
+			(xy 215.9 223.52) (xy 260.35 223.52)
 		)
 		(stroke
@@
 	(wire
 		(pts
-			(xy 219.71 238.76) (xy 219.71 251.46)
+			(xy 241.3 231.14) (xy 241.3 234.95)
 		)
 		(stroke
@@
 	(wire
 		(pts
-			(xy 203.2 255.27) (xy 203.2 257.81)
+			(xy 215.9 233.68) (xy 224.79 233.68)
 		)
 		(stroke
@@
 	(wire
 		(pts
-			(xy 215.9 223.52) (xy 260.35 223.52)
+			(xy 224.79 233.68) (xy 224.79 246.38)
 		)
 		(stroke
@@
 	(wire
 		(pts
-			(xy 241.3 231.14) (xy 241.3 234.95)
+			(xy 224.79 246.38) (xy 241.3 246.38)
 		)
 		(stroke
@@
 	(wire
 		(pts
-			(xy 215.9 233.68) (xy 224.79 233.68)
+			(xy 241.3 246.38) (xy 241.3 242.57)
 		)
 		(stroke
@@
 	(wire
 		(pts
-			(xy 224.79 233.68) (xy 224.79 246.38)
+			(xy 109.22 246.38) (xy 101.6 246.38)
 		)
 		(stroke
@@
 	(wire
 		(pts
-			(xy 224.79 246.38) (xy 241.3 246.38)
+			(xy 109.22 248.92) (xy 101.6 248.92)
 		)
 		(stroke
@@
 	(wire
 		(pts
-			(xy 241.3 246.38) (xy 241.3 242.57)
+			(xy 101.6 248.92) (xy 101.6 252.73)
 		)
 		(stroke
@@
 	(wire
 		(pts
-			(xy 109.22 246.38) (xy 101.6 246.38)
+			(xy 190.5 251.46) (xy 163.83 251.46)
 		)
 		(stroke
@@
 	(wire
 		(pts
-			(xy 109.22 248.92) (xy 101.6 248.92)
+			(xy 66.04 207.01) (xy 69.85 207.01)
 		)
 		(stroke
@@
 	(wire
 		(pts
-			(xy 101.6 248.92) (xy 101.6 252.73)
+			(xy 219.71 251.46) (xy 232.41 251.46)
 		)
 		(stroke
@@
 	)
 	(symbol
+		(lib_id "power:GND")
+		(at 228.6 236.22 0)
+		(unit 1)
+		(body_style 1)
+		(exclude_from_sim no)
+		(in_bom yes)
+		(on_board yes)
+		(in_pos_files yes)
+		(dnp no)
+		(property "Reference" "#PWR041"
+			(at 228.6 236.22 0)
+			(hide yes)
+			(show_name no)
+			(do_not_autoplace no)
+			(effects
+				(font
+					(size 1.27 1.27)
+				)
+			)
+		)
+		(property "Value" "GND"
+			(at 228.6 239.776 0)
+			(show_name no)
+			(do_not_autoplace no)
+			(effects
+				(font
+					(size 1.27 1.27)
+				)
+			)
+		)
+		(property "Footprint" ""
+			(at 228.6 236.22 0)
+			(hide yes)
+			(show_name no)
+			(do_not_autoplace no)
+			(effects
+				(font
+					(size 1.27 1.27)
+				)
+			)
+		)
+		(property "Datasheet" ""
+			(at 228.6 236.22 0)
+			(hide yes)
+			(show_name no)
+			(do_not_autoplace no)
+			(effects
+				(font
+					(size 1.27 1.27)
+				)
+			)
+		)
+		(property "Description" ""
+			(at 228.6 236.22 0)
+			(show_name no)
+			(do_not_autoplace no)
+			(effects
+				(font
+					(size 1.27 1.27)
+				)
+			)
+		)
+		(pin "1"
+		)
+		(instances
+			(project "kicad"
+				(path "/6c5b95c7-ee01-4343-9300-a46aa65ccf3e"
+					(reference "#PWR041")
+					(unit 1)
+				)
+			)
+		)
+	)
+	(symbol
 		(lib_id "Connector:USB_C_Receptacle_USB2.0_16P")
 		(at 44.45 60.96 0)
@@
 			)
 		)
-		(property "Footprint" "workshop:WSON-10-1EP_2x2mm_P0.4mm_EP0.9x1.5mm"
+		(property "Footprint" "Package_SON:WSON-10-1EP_2.5x2.5mm_P0.5mm_EP1.2x2mm"
 			(at 203.2 236.22 0)
 			(hide yes)
@@
 		)
 	)
-	(sheet_instances
-		(path "/"
-			(page "1")
-		)
-	)
-	(embedded_fonts no)
 	(symbol
 		(lib_id "Device:R")
@@
 	(symbol
 		(lib_id "power:GND")
-		(at 228.6 236.22 0)
+		(at 69.85 214.63 0)
 		(unit 1)
 		(body_style 1)
@@
 		(in_pos_files yes)
 		(dnp no)
-		(property "Reference" "#PWR041"
-			(at 228.6 236.22 0)
+		(property "Reference" "#PWR042"
+			(at 69.85 214.63 0)
 			(hide yes)
 			(show_name no)
@@
 		)
 		(property "Value" "GND"
-			(at 228.6 239.776 0)
+			(at 69.85 218.186 0)
 			(show_name no)
 			(do_not_autoplace no)
@@
 		)
 		(property "Footprint" ""
-			(at 228.6 236.22 0)
+			(at 69.85 214.63 0)
 			(hide yes)
 			(show_name no)
@@
 		)
 		(property "Datasheet" ""
-			(at 228.6 236.22 0)
+			(at 69.85 214.63 0)
 			(hide yes)
 			(show_name no)
@@
 		)
 		(property "Description" ""
-			(at 228.6 236.22 0)
+			(at 69.85 214.63 0)
 			(show_name no)
 			(do_not_autoplace no)
@@
 			(project "kicad"
 				(path "/6c5b95c7-ee01-4343-9300-a46aa65ccf3e"
-					(reference "#PWR041")
+					(reference "#PWR042")
 					(unit 1)
 				)
@@
 		)
 	)
-	(wire
-		(pts
-			(xy 219.71 251.46) (xy 232.41 251.46)
-		)
-		(stroke
-			(width 0)
-			(type default)
-		)
-	)
-	(no_connect
-		(at 50.8 218.44)
-	)
-	(junction
-		(at 66.04 207.01)
-		(diameter 0)
-		(color 0 0 0 0)
-	)
-	(wire
-		(pts
-			(xy 66.04 207.01) (xy 69.85 207.01)
-		)
-		(stroke
-			(width 0)
-			(type default)
-		)
-	)
 	(symbol
 		(lib_id "Device:R")
@@
 		)
 	)
-	(symbol
-		(lib_id "power:GND")
-		(at 69.85 214.63 0)
-		(unit 1)
-		(body_style 1)
-		(exclude_from_sim no)
-		(in_bom yes)
-		(on_board yes)
-		(in_pos_files yes)
-		(dnp no)
-		(property "Reference" "#PWR042"
-			(at 69.85 214.63 0)
-			(hide yes)
-			(show_name no)
-			(do_not_autoplace no)
-			(effects
-				(font
-					(size 1.27 1.27)
-				)
-			)
-		)
-		(property "Value" "GND"
-			(at 69.85 218.186 0)
-			(show_name no)
-			(do_not_autoplace no)
-			(effects
-				(font
-					(size 1.27 1.27)
-				)
-			)
-		)
-		(property "Footprint" ""
-			(at 69.85 214.63 0)
-			(hide yes)
-			(show_name no)
-			(do_not_autoplace no)
-			(effects
-				(font
-					(size 1.27 1.27)
-				)
-			)
-		)
-		(property "Datasheet" ""
-			(at 69.85 214.63 0)
-			(hide yes)
-			(show_name no)
-			(do_not_autoplace no)
-			(effects
-				(font
-					(size 1.27 1.27)
-				)
-			)
-		)
-		(property "Description" ""
-			(at 69.85 214.63 0)
-			(show_name no)
-			(do_not_autoplace no)
-			(effects
-				(font
-					(size 1.27 1.27)
-				)
-			)
-		)
-		(pin "1"
-		)
-		(instances
-			(project "kicad"
-				(path "/6c5b95c7-ee01-4343-9300-a46aa65ccf3e"
-					(reference "#PWR042")
-					(unit 1)
-				)
-			)
+	(sheet_instances
+		(path "/"
+			(page "1")
 		)
 	)
+	(embedded_fonts no)
 )

Commit message: workshop-5-1
Other:
- note removed: "NEO-PIXEL"
- note removed: "SCREEN"
Changed lines of the file:
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@@
-		)
-	)
-	(text "NEO-PIXEL"
-		(exclude_from_sim no)
-		(at 149.86 187.96 0)
-		(effects
-			(font
-				(size 6 6)
-			)
-			(justify left bottom)
 		)
 	)
@@
 		(effects
 			(font
-				(size 6 6)
-			)
-			(justify left bottom)
-		)
-	)
-	(text "SCREEN"
-		(exclude_from_sim no)
-		(at 285.75 201.93 0)
-		(effects
-			(font
